Commit message: 레이저 링크 및 조인트 이름을 'laser'로 변경

File: ros2_ws/src/robot_monitoring/urdf/myrobot.urdf.xacro (robot description, xacro)
@@ -63,5 +63,5 @@
     </joint>
     <!-- Laser -->
-    <link name="base_scan">
+    <link name="laser">
         <visual>
             <geometry>
@@ -74,7 +74,7 @@
         </visual>
     </link>
-    <joint name="base_link_to_base_scan" type="fixed">
+    <joint name="base_link_to_laser" type="fixed">
         <parent link="base_link"/>
-        <child link="base_scan"/>
+        <child link="laser"/>
         <origin xyz="${laser_x} ${laser_y} ${laser_z}" rpy="0 0 0"/>
     </joint>
